File: kicad/esp12e-oven/esp12e-oven.kicad_pcb (KiCad board)
At the start: 2 copper layers, 71.8 x 40 mm, 25 parts, among them P0 P0, P1 P2, P2 P3, P3 P1, P4 P5, P5 P4, P6 P6, P7 P7, U1 LM1117-3.3, U2 ESP-12E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

Commit message: Revised boards
Parts:
- added R3: 220K, Resistor_THT:R_Axial_DIN0204_L3.6mm_D1.6mm_P5.08mm_Horizontal, F.Cu at (66.7, 57.8)
- J2: renamed from I2C LCD
- P0: value P0 -> Probe 0
- P1: value P2 -> Probe 1
- P2: value P3 -> Probe 2
- P3: value P1 -> Probe 3
- P4: value P5 -> Probe 4
- P5: value P4 -> Probe 5
- P6: value P6 -> Probe 6
- P7: value P7 -> Probe 7
- RELAY0: renamed from RELAY1; value RELAY1 -> Relay 0
- RELAY1: renamed from RELAY0; value RELAY0 -> Relay 1
- moved P0 0.64 mm to (72.4, 68.6)
- moved P1 0.64 mm to (72.4, 62.9)
- moved R1 0.63 mm to (66.7, 40.0)
- moved R2 0.63 mm to (66.7, 48.9)
- renumbered DC to DC1, RESET to RESET1
Connections:
- U3 pad 3: Net-(R1-Pad1) -> Net-(R3-Pad1)
Routing:
- net Net-(C2-Pad1): track 150.4 -> 127.0 mm
- net Net-(R3-Pad1): track 0.00 -> 17.8 mm
- net Net-(R1-Pad1): track 54.5 -> 38.6 mm
- net Net-(P0-Pad1): track 19.7 -> 27.7 mm
- net Net-(P7-Pad1): track 38.4 -> 41.7 mm
- net Net-(RELAY1-Pad2): track 56.0 -> 58.9 mm
- net Net-(P6-Pad1): track 42.5 -> 44.8 mm
- net Net-(P1-Pad1): track 21.4 -> 19.5 mm
- net Net-(P2-Pad1): track 34.5 -> 32.7 mm
- net Net-(C1-Pad1): track 144.8 -> 146.0 mm
- net Net-(RELAY0-Pad2): track 48.4 -> 47.3 mm
- net Net-(P5-Pad1): track 32.3 -> 33.1 mm
- net Net-(C1-Pad2): track 42.3 -> 42.8 mm
